File: oresat-diode-test-card/oresat-diode-test-card.kicad_pcb (KiCad board)
At the start: 4 copper layers, 99.8 x 94.6 mm, 138 parts, among them J6 J-SAMTEC-TFM-120-X1-XXX-D-RA, J7 ORESAT-DEBUG-CONNECTOR-ALL, Q1 DMP2240UDM, Q2 DMP3050LVT-7, Q3 NMOS, Q4 DMP3050LVT-7, Q7 MOSFET-PCH-SOT23-6, Q8 PMV45EN, Q9 PMV45EN, U1 TCAN330, U10 TPS62111RSA, U11 MIC842LYC5, U12 MIC842LYC5, U2 MAX7310, U3 TS5A21366DCUR, U4 TLV6001DCK, U501 TLV6001DCK, U6 MAX4211, U7 STM32F091C, U8 NX3L4051-Q100, U9 TLV6001DCK, X2 CRYSTAL-WITH-GND

Commit message: another layout rev
Parts:
- added REF**: SWIR Diode Cover, oresat-diodes:SWIR Diode Cover, F.Cu at (162.9, 104.3)
- added REF**: SWIR Diode Cover, oresat-diodes:SWIR Diode Cover, F.Cu at (162.9, 130.3)
- moved U9 16.3 mm to (156.2, 102.3)
- moved U5 15.4 mm to (162.9, 104.8), turned to 90 degrees
- moved C12 15.0 mm to (156.0, 104.5), turned to 180 degrees
- moved R10 14.8 mm to (137.5, 107.4), turned to 0 degrees
- moved C10 13.0 mm to (156.2, 100.3), turned to 0 degrees
- moved R14 11.8 mm to (156.2, 99.2), turned to 180 degrees
- moved U4 11.1 mm to (138.9, 105.2)
- moved C7 10.9 mm to (140.3, 108.6), turned to 0 degrees
- moved R12 10.8 mm to (136.8, 104.8), turned to -90 degrees
- moved R11 9.55 mm to (140.3, 107.4), turned to 180 degrees
- moved U8 4.80 mm to (143.4, 115.4)
- moved D8 3.74 mm to (162.3, 130.3), turned to 90 degrees
- moved D1 2.79 mm to (160.2, 125.2)
- moved Q3 2.76 mm to (144.8, 102.4), turned to 0 degrees
- moved R501 2.49 mm to (157.5, 128.9)
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Routing:
- net 3.3V: track 119.1 -> 10.2 mm, vias 16 -> 13
- net Net-(D1-A): track 85.7 -> 0.00 mm, vias 4 -> 0
- net Net-(U5-1460nm): track 48.6 -> 0.00 mm, vias 2 -> 0
- net Net-(U5-1040nm): track 46.3 -> 0.00 mm, vias 2 -> 0
- net Net-(U5-1200nm): track 44.8 -> 0.00 mm, vias 2 -> 0
- net Net-(U5-1300nm): track 44.6 -> 0.00 mm, vias 2 -> 0
- net Net-(U5-1550nm): track 38.0 -> 0.00 mm, vias 2 -> 0
- net LED_CURRENT: track 79.6 -> 61.8 mm, vias 4 -> 2
- net SWIR_PD_CURRENT: track 85.5 -> 68.9 mm
- net Net-(D2-K): track 21.9 -> 9.52 mm
- net Net-(Q3-G): track 16.3 -> 5.43 mm
- net Net-(D4-K): track 21.1 -> 11.2 mm
- net Net-(U5-PD_Cathode): track 8.53 -> 0.00 mm
- net DAC_OUT: track 56.8 -> 48.7 mm
- net Net-(Q4-D-Pad1): track 17.1 -> 10.2 mm
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