File: oresat-diode-test-card/oresat-diode-test-card.kicad_sch (KiCad schematic)
At the start: 0 parts

Commit message: added actual files
Other:
- added sheet SWIR Diode (oresat-diode-test-card-sch-SWIR.kicad_sch)
Changed lines of the file:
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@@
+	)
+	(sheet
+		(at 190.5 149.86)
+		(size 12.7 3.81)
+		(fields_autoplaced yes)
+		(stroke
+			(width 0.1524)
+			(type solid)
+		)
+		(fill
+			(color 0 0 0 0.0000)
+		)
+		(property "Sheetname" "SWIR Diode"
+			(at 190.5 149.1484 0)
+			(effects
+				(font
+					(size 1.27 1.27)
+				)
+				(justify left bottom)
+			)
+		)
+		(property "Sheetfile" "oresat-diode-test-card-sch-SWIR.kicad_sch"
+			(at 190.5 154.2546 0)
+			(effects
+				(font
+					(size 1.27 1.27)
+				)
+				(justify left top)
+			)
+		)
+		(property "Field2" ""
+			(at 190.5 149.86 0)
+			(effects
+				(font
+					(size 1.27 1.27)
+				)
+				(hide yes)
+			)
+		)
+		(instances
+			(project "oresat-diode-test-card"
+				(path "/04d32576-d084-475b-9eac-d7f3fd9579d7"
+					(page "5")
+				)
+			)
+		)
 	)
 	(sheet

Commit message: Quick design review on schematic; basically ready for layout.
Other:
- title: OreSat M0 Proto Card -> OreSat Diode Test Card
Changed lines of the file:
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@@
 	(paper "USLedger")
 	(title_block
-		(title "OreSat M0 Proto Card")
-		(date "2024-03-21")
-		(rev "5.0")
+		(title "OreSat Diode Test Card")
+		(date "2024-04-21")
+		(rev "v1.0")
 	)
 	(sheet
